File: pcb/demoCurrentSensor.kicad_sch (KiCad schematic)
At the start: 16 parts

Commit message: PCB design progress
Parts:
- 3.3, IO0, RXD0, TXD0: footprint SymbioteFootprints:TestPointLarge -> TestPoint:TestPoint_Pad_D1.5mm
- BT1: renamed from BT?; footprint (none) -> KiCadGlobal:BatteryHolder_Keystone_2466_1xAAA
- C1, C2: renamed from C?; footprint Capacitors_SMD:C_0805 -> Capacitor_SMD:C_0805_2012Metric
- C3, C4: renamed from C?; footprint Capacitors_SMD:C_0805 -> Capacitor_SMD:C_0603_1608Metric
- EN1: renamed from EN; footprint SymbioteFootprints:TestPointLarge -> TestPoint:TestPoint_Pad_D1.5mm
- GND1: renamed from GND; footprint SymbioteFootprints:TestPointLarge -> TestPoint:TestPoint_Pad_D1.5mm
- L1: renamed from L?; footprint (none) -> Inductor_SMD:L_Bourns-SRN4018
- R1: renamed from R?; footprint (none) -> Resistor_SMD:R_0603_1608Metric
- U1: renamed from U?; footprint (none) -> Package_TO_SOT_SMD:SOT-23
- U2: renamed from U?; footprint (none) -> KiCadGlobal:SOIC-8-1EP_3.9x4.9mm_P1.27mm
- U3: renamed from U?; footprint SymbioteFootprints:ESP32-WROOM-32E -> KiCadGlobal:ESP32-WROOM-32E
Connections:
- net 3.3: now reaches 3.3.1, C1.1, C2.1, C3.1, C4.2, R1.1, U1.1 (3.3), U2.1 (VSUP), U3.2 (3V3)
- net GND: now reaches BT1.2 (-), C1.2, C2.2, C3.2, C4.1, GND1.1, U1.3 (GND), U2.2 (GND), U2.3 (Test), U3.1 (GND), U3.15 (GND), U3.38 (GND), U3.39 (GND)
