File: pcb/demoCurrentSensor.kicad_pcb (KiCad board)
At the start: 2 copper layers, 50 x 28 mm, 16 parts, among them U1 TPS613221A, U2 Cur4000, U3 ESP32-WROOM

Commit message: PCB routing
Parts:
- moved TXD0 9.66 mm to (22.0, -19.0), turned to 0 degrees
- moved 3.3 8.46 mm to (18.0, -15.0), turned to 0 degrees
- moved GND1 8.46 mm to (18.0, -19.0), turned to 0 degrees
- moved IO0 7.13 mm to (22.0, -11.0), turned to 0 degrees
- moved RXD0 2.91 mm to (22.0, -15.0), turned to 0 degrees
- moved EN1 2.91 mm to (18.0, -11.0), turned to 0 degrees
- moved U2 0.27 mm to (3.50, -19.9)
- moved R1 0.18 mm to (19.5, -2.83)
Routing:
- net /3.3: track 0.00 -> 46.4 mm, vias 0 -> 2
- net Net-(U2-Pad4): track 0.00 -> 43.3 mm
- net Net-(U2-Pad7): track 0.00 -> 38.1 mm, vias 0 -> 2
- net Net-(U2-Pad5): track 0.00 -> 36.9 mm, vias 0 -> 2
- net Net-(U2-Pad8): track 0.00 -> 33.7 mm
- net Net-(U2-Pad6): track 0.00 -> 29.9 mm
- net Net-(IO0-Pad1): track 0.00 -> 27.3 mm, vias 0 -> 2
- net Net-(TXD0-Pad1): track 0.00 -> 23.8 mm, vias 0 -> 2
- net Net-(RXD0-Pad1): track 0.00 -> 23.1 mm, vias 0 -> 2
- net Net-(EN1-Pad1): track 0.00 -> 21.1 mm, vias 0 -> 2
- net Net-(BT1-Pad1): track 1.74 -> 0.00 mm
- net /GND: vias 0 -> 68
- added copper zone on B.Cu, net /GND
- added copper zone on F.Cu, net /GND
- added copper zone on F.Cu, net Net-(BT1-Pad1)
- added copper zone on F.Cu, net Net-(L1-Pad2)

Commit message: tuning solidworks
Parts:
- moved U3 0.67 mm to (36.0, -15.0)
- moved U2 0.39 mm to (3.13, -20.0)
- moved L1 0.30 mm to (7.00, -3.00)
Routing:
- net Net-(U2-Pad7): track 38.1 -> 39.5 mm
- net Net-(U2-Pad4): track 43.3 -> 42.4 mm
- net Net-(EN1-Pad1): track 21.1 -> 21.9 mm
- net Net-(IO0-Pad1): track 27.3 -> 26.4 mm
- net /3.3: track 46.4 -> 47.2 mm
- net /GND: vias 68 -> 65
